Commit message: modify file position

File: s4_gun/urdf/gun.urdf.xacro (robot description, xacro)
@@ -11,5 +11,5 @@
         <origin xyz="0 0 0" rpy="0 0 0"/>
         <geometry>
-          <mesh filename="package://srs004host/urdf/base1.stl" />
+          <mesh filename="package://s4_gun/stl/base1.stl" />
         </geometry>
         <material name="gray"/>
@@ -31,5 +31,5 @@
         <origin xyz="0 0 0" rpy="0 0 0"/>
         <geometry>
-          <mesh filename="package://srs004host/urdf/base2.stl" />
+          <mesh filename="package://s4_gun/stl/base2.stl" />
         </geometry>
         <material name="gray"/>
@@ -51,5 +51,5 @@
         <origin xyz="0 0 0" rpy="0 0 0"/>
         <geometry>
-          <mesh filename="package://srs004host/urdf/gun.stl" />
+          <mesh filename="package://s4_gun/stl/gun.stl" />
         </geometry>
         <material name="light_red"/>

File: s4_omni/urdf/wheel.urdf.xacro (robot description, xacro)
@@ -2,5 +2,5 @@
 <robot xmlns:xacro="http://ros.org/wiki/xacro">
   <xacro:macro name="barrel" params="prefix parent dir">
-    <joint name="${prefix}_joint" type="continuous">
+    <joint name="${prefix}_joint" type="fixed"><!--continuous-->
       <parent link="${parent}"/>
       <child link="${prefix}_link"/>
@@ -26,4 +26,5 @@
       </inertial>
     </link>
+<!--
     <joint name="${prefix}_mark_joint" type="fixed">
       <parent link="${prefix}_link"/>
@@ -43,4 +44,5 @@
       </inertial>
     </link>
+-->
     <!-- ===============  Gazebo =============== -->
     <gazebo reference="${prefix}_link">

File: s4_omni/urdf/world.urdf.xacro (robot description, xacro)
@@ -9,4 +9,9 @@
     <child link="base_link"/>
   </joint>
+  <link name="target/t1"/>
+  <joint name="target/t1_joint" type="fixed">
+    <parent link="world"/>
+    <child link="target/t1"/>
+  </joint>
   <xacro:s4_omni prefix="body0" parent="base_link" />
   <!-- ===============  Gazebo =============== -->

Commit message: change gun name

File: s4_gun/urdf/gun.urdf.xacro (robot description, xacro)
@@ -2,10 +2,10 @@
 <robot xmlns:xacro="http://ros.org/wiki/xacro">
   <xacro:macro name="gun_tullet" params="prefix parent pos_x pos_z">
-    <joint name="${prefix}_base1_joint" type="fixed">
+    <joint name="${prefix}/base1_joint" type="fixed">
       <parent link="${parent}"/>
-      <child link="${prefix}_base1_link"/>
+      <child link="${prefix}/base1_link"/>
       <origin rpy="0 0 0" xyz="${pos_x} 0 ${pos_z}"/>
     </joint>
-    <link name="${prefix}_base1_link">
+    <link name="${prefix}/base1_link">
       <visual>
         <origin xyz="0 0 0" rpy="0 0 0"/>
@@ -20,12 +20,12 @@
       </inertial>
     </link>
-    <joint name="${prefix}_base2_joint" type="continuous">
-      <parent link="${prefix}_base1_link"/>
-      <child link="${prefix}_base2_link"/>
+    <joint name="${prefix}/base2_joint" type="continuous">
+      <parent link="${prefix}/base1_link"/>
+      <child link="${prefix}/base2_link"/>
       <origin rpy="0 0 0" xyz="0 0 0.016"/>
       <axis xyz="0 0 1"/>
       <dynamics damping="0.7"/>
     </joint>
-    <link name="${prefix}_base2_link">
+    <link name="${prefix}/base2_link">
       <visual>
         <origin xyz="0 0 0" rpy="0 0 0"/>
@@ -40,12 +40,12 @@
       </inertial>
     </link>
-    <joint name="${prefix}_gun_joint" type="continuous">
-      <parent link="${prefix}_base2_link"/>
-      <child link="${prefix}_gun_link"/>
+    <joint name="${prefix}/gun_joint" type="continuous">
+      <parent link="${prefix}/base2_link"/>
+      <child link="${prefix}/gun_link"/>
       <origin rpy="0 0 0" xyz="0 0 0.070"/>
       <axis xyz="0 1 0"/>
       <dynamics damping="0.1"/>
     </joint>
-    <link name="${prefix}_gun_link">
+    <link name="${prefix}/gun_link">
       <visual>
         <origin xyz="0 0 0" rpy="0 0 0"/>

File: s4_gun/urdf/world.urdf.xacro (robot description, xacro)
@@ -4,10 +4,10 @@
   <xacro:include filename="$(find s4_gun)/urdf/gun.urdf.xacro"/>
   <link name="world"/>
-  <link name="base_link"/>
-  <joint name="base_joint" type="fixed"><!--floating-->
+  <link name="robot0/base_link"/>
+  <joint name="robot0/base_joint" type="fixed"><!--floating-->
     <parent link="world"/>
-    <child link="base_link"/>
+    <child link="robot0/base_link"/>
   </joint>
-  <xacro:gun_tullet prefix="gun0" parent="base_link" pos_x="0.010" pos_z="0.038" />
+  <xacro:gun_tullet prefix="robot0/gun0" parent="robot0/base_link" pos_x="0.010" pos_z="0.038" />
   <!-- ===============  Gazebo =============== -->
   <gazebo>
