Commit message: modify urdf and stl

File: s4_gun/urdf/common.urdf.xacro (robot description, xacro)
@@ -17,6 +17,12 @@
     <color rgba="1.0 0.5 0.5 2.5"/>
   </material>
-  <material name="yellow">
-    <color rgba="0 1.0 1.0 2.5"/>
+  <material name="green">
+    <color rgba="0 1.0 0 2.5"/>
+  </material>
+  <material name="blue">
+    <color rgba="0 0 1.0 2.5"/>
+  </material>
+  <material name="wood">
+    <color rgba="0.9 0.9 0.5 2.5"/>
   </material>
 </robot>

File: s4_launch/urdf/common.urdf.xacro (robot description, xacro)
@@ -17,12 +17,15 @@
     <color rgba="1.0 0.5 0.5 2.5"/>
   </material>
-  <material name="yellow">
-    <color rgba="1.0 1.0 0.0 2.5"/>
-  </material>
   <material name="green">
-    <color rgba="0.0 1.0 0 2.5"/>
+    <color rgba="0 1.0 0 2.5"/>
   </material>
   <material name="dark_green">
-    <color rgba="0.0 0.5 0 2.5"/>
+    <color rgba="0 0.5 0 2.5"/>
+  </material>
+  <material name="blue">
+    <color rgba="0 0 1.0 2.5"/>
+  </material>
+  <material name="wood">
+    <color rgba="0.9 0.9 0.5 2.5"/>
   </material>
 </robot>

File: s4_launch/urdf/s4_robot.urdf.xacro (robot description, xacro)
@@ -11,8 +11,8 @@
       <child link="${prefix}/base_link"/>
     </joint>
-    <xacro:s4_body      prefix="${prefix}/body0"      parent="${prefix}/base_link" pos_z="0.041"/>
+    <xacro:s4_body      prefix="${prefix}/body0"      parent="${prefix}/base_link" pos_z="0.044"/>
     <xacro:s4_omni      prefix="${prefix}/omni0"      parent="${prefix}/base_link" />
-    <xacro:s4_gun       prefix="${prefix}/gun0"       parent="${prefix}/base_link" pos_x="0.0" pos_z="0.079" />
-    <xacro:s4_hitsensor prefix="${prefix}/hitsensor0" parent="${prefix}/base_link" radius="0.106" height="0.079" />
+    <xacro:s4_gun       prefix="${prefix}/gun0"       parent="${prefix}/base_link" pos_x="0.020" pos_z="0.082" />
+    <xacro:s4_hitsensor prefix="${prefix}/hitsensor0" parent="${prefix}/base_link" radius="0.106" height="0.082" />
   </xacro:macro>
   <!-- ===============  Gazebo =============== -->

File: s4_omni/urdf/s4_omni.urdf.xacro (robot description, xacro)
@@ -3,7 +3,7 @@
   <xacro:include filename="$(find s4_omni)/urdf/wheel.urdf.xacro"/>
   <xacro:macro name="s4_omni" params="prefix parent">
-    <xacro:omni_wheel prefix="${prefix}/wheel0" parent="${parent}" radius="0.075" dir="${pi/3}"   height="0.019" />
-    <xacro:omni_wheel prefix="${prefix}/wheel1" parent="${parent}" radius="0.075" dir="${pi}"     height="0.019" />
-    <xacro:omni_wheel prefix="${prefix}/wheel2" parent="${parent}" radius="0.075" dir="${5*pi/3}" height="0.019" />
+    <xacro:omni_wheel prefix="${prefix}/wheel0" parent="${parent}" radius="0.077" dir="${pi/3}"   height="0.019" />
+    <xacro:omni_wheel prefix="${prefix}/wheel1" parent="${parent}" radius="0.077" dir="${pi}"     height="0.019" />
+    <xacro:omni_wheel prefix="${prefix}/wheel2" parent="${parent}" radius="0.077" dir="${5*pi/3}" height="0.019" />
   </xacro:macro>
   <!-- ===============  Gazebo =============== -->

File: s4_omni/urdf/wheel.urdf.xacro (robot description, xacro)
@@ -26,23 +26,4 @@
       </inertial>
     </link>
-<!--
-    <joint name="${prefix}_mark_joint" type="fixed">
-      <parent link="${prefix}_link"/>
-      <child link="${prefix}_mark_link"/>
-      <origin rpy="0 0 0" xyz="0.005 0 0"/>
-    </joint>
-    <link name="${prefix}_mark_link">
-      <visual>
-        <geometry>
-          <box size="0.005 0.005 0.005"/>
-        </geometry>
-        <material name="white"/>
-      </visual>
-      <inertial>
-        <mass value="0.001"/>
-        <inertia ixx="0.0001" ixy="0" ixz="0" iyy="0.0001" iyz="0" izz="0.0001"/>
-      </inertial>
-    </link>
--->
     <!-- ===============  Gazebo =============== -->
     <gazebo reference="${prefix}_link">
@@ -59,5 +40,5 @@
       <parent link="${parent}"/>
       <child link="${prefix}/motor_link"/>
-      <origin rpy="0 ${pi/2} ${dir}" xyz="${radius*cos(dir)} ${radius*sin(dir)} ${height}"/>
+      <origin rpy="0 0 ${dir}" xyz="${radius*cos(dir)} ${radius*sin(dir)} ${height}"/>
     </joint>
     <link name="${prefix}/motor_link">
@@ -65,4 +46,22 @@
         <geometry>
           <mesh filename="package://s4_omni/stl/motor.stl" />
+        </geometry>
+        <origin xyz="0 0 0" rpy="0 0 0"/>
+        <material name="gray"/>
+      </visual>
+      <inertial>
+        <mass value="0.180"/>
+        <inertia ixx="0.0001" ixy="0" ixz="0" iyy="0.0001" iyz="0" izz="0.0001"/>
+      </inertial>
+    </link>
+    <joint name="${prefix}/motor_mount_joint" type="fixed">
+      <parent link="${parent}"/>
+      <child link="${prefix}/motor_mount_link"/>
+      <origin rpy="0 0 ${dir}" xyz="${radius*cos(dir)} ${radius*sin(dir)} ${height}"/>
+    </joint>
+    <link name="${prefix}/motor_mount_link">
+      <visual>
+        <geometry>
+          <mesh filename="package://s4_omni/stl/motor_mounter.stl" />
         </geometry>
         <origin xyz="0 0 0" rpy="0 0 0"/>

File: s4_operate/urdf/s4_body.urdf.xacro (robot description, xacro)
@@ -20,8 +20,26 @@
       </inertial>
     </link>
+    <joint name="${prefix}/battery_joint" type="fixed">
+      <parent link="${prefix}/body_link"/>
+      <child  link="${prefix}/battery_link"/>
+      <origin rpy="0 0 0" xyz="0.065 0 0.004"/>
+    </joint>
+    <link name="${prefix}/battery_link">
+      <visual>
+        <origin xyz="0 0 0" rpy="0 0 0"/>
+        <geometry>
+          <mesh filename="package://s4_operate/stl/battery.stl" />
+        </geometry>
+        <material name="blue"/>
+      </visual>
+      <inertial>
+        <mass value="0.130"/>
+        <inertia ixx="0.0001" ixy="0" ixz="0" iyy="0.0001" iyz="0" izz="0.0001"/>
+      </inertial>
+    </link>
     <joint name="${prefix}/bridge_joint" type="fixed">
       <parent link="${prefix}/body_link"/>
       <child  link="${prefix}/bridge_link"/>
-      <origin rpy="0 0 0" xyz="0 0 0.182"/>
+      <origin rpy="0 0 0" xyz="0.005 0 0.183"/>
     </joint>
     <link name="${prefix}/bridge_link">
@@ -38,4 +56,22 @@
       </inertial>
     </link>
+    <joint name="${prefix}/camera_joint" type="fixed">
+      <parent link="${prefix}/bridge_link"/>
+      <child  link="${prefix}/camera_link"/>
+      <origin rpy="-1.5707 0 -1.5707" xyz="0.015 0 0.019"/>
+    </joint>
+    <link name="${prefix}/camera_link">
+      <visual>
+        <origin xyz="0 0 0" rpy="0 0 0"/>
+        <geometry>
+          <mesh filename="package://s4_operate/stl/camera.stl" />
+        </geometry>
+        <material name="light_red"/>
+      </visual>
+      <inertial>
+        <mass value="0.190"/>
+        <inertia ixx="0.001" ixy="0" ixz="0" iyy="0.001" iyz="0" izz="0.0001"/>
+      </inertial>
+    </link>
   </xacro:macro>
 </robot>

File: s4_vive/urdf/s4_vive.urdf.xacro (robot description, xacro)
@@ -40,5 +40,5 @@
     <link name="${prefix}/body_link">
       <visual>
-        <origin rpy="0 0 0" xyz="0 0 0"/>
+        <origin rpy="0 0 0" xyz="-0.005 0 0"/>
         <geometry>
           <mesh filename="package://s4_vive/stl/vive_tracker.stl"/>
@@ -60,5 +60,5 @@
       <parent link="${prefix}/body_link"/>
       <child  link="${prefix}/tracking_link"/>
-      <origin xyz="-0.265 -0.025 0.050" rpy="-1.5707 0 -1.5707"/>
+      <origin xyz="-0.271 -0.025 0.050" rpy="-1.5707 0 -1.5707"/>
     </joint>
   </xacro:macro>
