Commit message: modify launch

File: s4_gun/urdf/s4_gun.urdf.xacro (robot description, xacro)
@@ -1,5 +1,5 @@
 <?xml version="1.0"?>
 <robot xmlns:xacro="http://ros.org/wiki/xacro">
-  <xacro:macro name="gun_tullet" params="prefix parent pos_x pos_z">
+  <xacro:macro name="s4_gun" params="prefix parent pos_x pos_z">
     <joint name="${prefix}/base1_joint" type="fixed">
       <parent link="${parent}"/>

File: s4_gun/urdf/world.urdf.xacro (robot description, xacro)
@@ -2,5 +2,5 @@
 <robot name="my_robo" xmlns:xacro="http://ros.org/wiki/xacro">
   <xacro:include filename="$(find s4_gun)/urdf/common.urdf.xacro"/>
-  <xacro:include filename="$(find s4_gun)/urdf/gun.urdf.xacro"/>
+  <xacro:include filename="$(find s4_gun)/urdf/s4_gun.urdf.xacro"/>
   <link name="world"/>
   <link name="robot0/base_link"/>
@@ -9,5 +9,5 @@
     <child link="robot0/base_link"/>
   </joint>
-  <xacro:gun_tullet prefix="robot0/gun0" parent="robot0/base_link" pos_x="0.010" pos_z="0.038" />
+  <xacro:s4_gun prefix="robot0/gun0" parent="robot0/base_link" pos_x="0.010" pos_z="0.038" />
   <!-- ===============  Gazebo =============== -->
   <gazebo>

File: s4_hitsensor/urdf/s4_hitsensor.urdf.xacro (robot description, xacro)
@@ -1,5 +1,5 @@
 <?xml version="1.0"?>
 <robot xmlns:xacro="http://ros.org/wiki/xacro">
-  <xacro:macro name="hitsensor" params="prefix parent xyz rpy">
+  <xacro:macro name="s4_target" params="prefix parent xyz rpy">
     <link name="${prefix}/frame_link">
       <visual>
@@ -31,3 +31,8 @@
     </joint>
   </xacro:macro>
+  <xacro:macro name="s4_hitsensor" params="prefix parent radius height">
+    <xacro:s4_target  prefix="${prefix}/target0" parent="${parent}" xyz="${radius*cos(pi/3)}   ${radius*sin(pi/3)} ${height}"   rpy="0 0 ${pi/3}" />
+    <xacro:s4_target  prefix="${prefix}/target1" parent="${parent}" xyz="${radius*cos(pi)}     ${radius*sin(pi)} ${height}"     rpy="0 0 ${pi}" />
+    <xacro:s4_target  prefix="${prefix}/target2" parent="${parent}" xyz="${radius*cos(5*pi/3)} ${radius*sin(5*pi/3)} ${height}" rpy="0 0 ${5*pi/3}" />
+  </xacro:macro>
 </robot>

File: s4_hitsensor/urdf/world.urdf.xacro (robot description, xacro)
@@ -5,11 +5,9 @@
   <link name="world"/>
   <link name="robot0/base_link"/>
-  <joint name="robot0/base_joint" type="fixed"><!--floating-->
+  <joint name="robot0/base_joint" type="fixed">
     <parent link="world"/>
     <child link="robot0/base_link"/>
   </joint>
-  <xacro:hitsensor prefix="robot0/hitsensor/target0" parent="robot0/base_link" xyz=" 0.05  0.07 0" rpy="0 0 ${pi/3}" />
-  <xacro:hitsensor prefix="robot0/hitsensor/target1" parent="robot0/base_link" xyz="-0.10  0    0" rpy="0 0 ${pi}" />
-  <xacro:hitsensor prefix="robot0/hitsensor/target2" parent="robot0/base_link" xyz=" 0.05 -0.07 0" rpy="0 0 ${5*pi/3}" />
+  <xacro:s4_hitsensor prefix="robot0/hitsensor0" parent="robot0/base_link" radius="0.1" height="0.1" />
   <!-- ===============  Gazebo =============== -->
   <gazebo>

Commit message: s4_gun:refactoring

File: s4_gun/urdf/s4_gun.urdf.xacro (robot description, xacro)
@@ -60,4 +60,10 @@
       </inertial>
     </link>
+    <joint name="${prefix}/laser_joint" type="fixed">
+      <parent link="${prefix}/gun_link"/>
+      <child link="${prefix}/laser_link"/>
+      <origin rpy="0 0 0" xyz="0.030 0 -0.034"/>
+    </joint>
+    <link name="${prefix}/laser_link"/>
     <!-- ===============  Transmission =============== -->
     <transmission name="${prefix}_base2_trans">

Commit message: s4_comport: add remote1,2 s4_gun: add target mode

File: s4_gun/urdf/s4_gun.urdf.xacro (robot description, xacro)
@@ -66,4 +66,10 @@
     </joint>
     <link name="${prefix}/laser_link"/>
+    <joint name="${prefix}/standard_joint" type="fixed">
+      <parent link="${parent}"/>
+      <child link="${prefix}/gun_standard"/>
+      <origin rpy="0 0 0" xyz="0.01 0 0.124"/>
+    </joint>
+    <link name="${prefix}/gun_standard" />
     <!-- ===============  Transmission =============== -->
     <transmission name="${prefix}_base2_trans">
