Commit message: change omni name

File: s4_omni/urdf/s4_omni.urdf.xacro (robot description, xacro)
@@ -14,7 +14,7 @@
     <xacro:body prefix="body0" parent="base_link" />
 -->
-    <xacro:omni_wheel prefix="wheel0" parent="base_link" radius="0.075" dir="${pi/3}"   height="-0.022" />
-    <xacro:omni_wheel prefix="wheel1" parent="base_link" radius="0.075" dir="${pi}"     height="-0.022" />
-    <xacro:omni_wheel prefix="wheel2" parent="base_link" radius="0.075" dir="${5*pi/3}" height="-0.022" />
+    <xacro:omni_wheel prefix="${prefix}/wheel0" parent="${parent}" radius="0.075" dir="${pi/3}"   height="0.019" />
+    <xacro:omni_wheel prefix="${prefix}/wheel1" parent="${parent}" radius="0.075" dir="${pi}"     height="0.019" />
+    <xacro:omni_wheel prefix="${prefix}/wheel2" parent="${parent}" radius="0.075" dir="${5*pi/3}" height="0.019" />
   </xacro:macro>
   <!-- ===============  Gazebo =============== -->

File: s4_omni/urdf/wheel.urdf.xacro (robot description, xacro)
@@ -56,10 +56,10 @@
   </xacro:macro>
   <xacro:macro name="omni_wheel" params="prefix parent radius dir height">
-    <joint name="${prefix}_motor_joint" type="fixed">
+    <joint name="${prefix}/motor_joint" type="fixed">
       <parent link="${parent}"/>
-      <child link="${prefix}_motor_link"/>
+      <child link="${prefix}/motor_link"/>
       <origin rpy="0 ${pi/2} ${dir}" xyz="${radius*cos(dir)} ${radius*sin(dir)} ${height}"/>
     </joint>
-    <link name="${prefix}_motor_link">
+    <link name="${prefix}/motor_link">
       <visual>
         <geometry>
@@ -74,12 +74,12 @@
       </inertial>
     </link>
-    <joint name="${prefix}_housing_joint" type="continuous">
+    <joint name="${prefix}/housing_joint" type="continuous">
       <parent link="${parent}"/>
-      <child link="${prefix}_housing_link"/>
+      <child link="${prefix}/housing_link"/>
       <origin rpy="0 ${pi/2} ${dir}" xyz="${(radius+0.0222)*cos(dir)} ${(radius+0.0222)*sin(dir)} ${height}"/>
       <axis xyz="0 0 1"/>
       <dynamics damping="0.1"/>
     </joint>
-    <link name="${prefix}_housing_link">
+    <link name="${prefix}/housing_link">
       <visual>
         <geometry>
@@ -94,10 +94,10 @@
       </inertial>
     </link>
-    <joint name="${prefix}_housing_s_joint" type="fixed">
-      <parent link="${prefix}_housing_link"/>
-      <child link="${prefix}_housing_s_link"/>
+    <joint name="${prefix}/housing_s_joint" type="fixed">
+      <parent link="${prefix}/housing_link"/>
+      <child link="${prefix}/housing_s_link"/>
       <origin rpy="0 ${pi} ${pi/4}" xyz="0 0 0"/>
     </joint>
-    <link name="${prefix}_housing_s_link">
+    <link name="${prefix}/housing_s_link">
       <inertial>
         <mass value="0.001"/>
@@ -105,12 +105,12 @@
       </inertial>
     </link>
-    <xacro:barrel prefix="${prefix}_barrel_1" parent="${prefix}_housing_link" dir="0"/>
-    <xacro:barrel prefix="${prefix}_barrel_2" parent="${prefix}_housing_link" dir="${pi/2}"/>
-    <xacro:barrel prefix="${prefix}_barrel_3" parent="${prefix}_housing_link" dir="${pi}"/>
-    <xacro:barrel prefix="${prefix}_barrel_4" parent="${prefix}_housing_link" dir="${-pi/2}"/>
-    <xacro:barrel prefix="${prefix}_barrel_5" parent="${prefix}_housing_s_link" dir="0"/>
-    <xacro:barrel prefix="${prefix}_barrel_6" parent="${prefix}_housing_s_link" dir="${pi/2}"/>
-    <xacro:barrel prefix="${prefix}_barrel_7" parent="${prefix}_housing_s_link" dir="${pi}"/>
-    <xacro:barrel prefix="${prefix}_barrel_8" parent="${prefix}_housing_s_link" dir="${-pi/2}"/>
+    <xacro:barrel prefix="${prefix}/barrel_1" parent="${prefix}/housing_link" dir="0"/>
+    <xacro:barrel prefix="${prefix}/barrel_2" parent="${prefix}/housing_link" dir="${pi/2}"/>
+    <xacro:barrel prefix="${prefix}/barrel_3" parent="${prefix}/housing_link" dir="${pi}"/>
+    <xacro:barrel prefix="${prefix}/barrel_4" parent="${prefix}/housing_link" dir="${-pi/2}"/>
+    <xacro:barrel prefix="${prefix}/barrel_5" parent="${prefix}/housing_s_link" dir="0"/>
+    <xacro:barrel prefix="${prefix}/barrel_6" parent="${prefix}/housing_s_link" dir="${pi/2}"/>
+    <xacro:barrel prefix="${prefix}/barrel_7" parent="${prefix}/housing_s_link" dir="${pi}"/>
+    <xacro:barrel prefix="${prefix}/barrel_8" parent="${prefix}/housing_s_link" dir="${-pi/2}"/>
     <!-- ===============  Transmission =============== -->
     <transmission name="${prefix}_housing_trans">

File: s4_omni/urdf/world.urdf.xacro (robot description, xacro)
@@ -4,15 +4,10 @@
   <xacro:include filename="$(find s4_omni)/urdf/s4_omni.urdf.xacro"/>
   <link name="world"/>
-  <link name="base_link"/>
-  <joint name="base_joint" type="floating">
+  <link name="robot0/base_link"/>
+  <joint name="robot0/base_joint" type="floating">
     <parent link="world"/>
-    <child link="base_link"/>
+    <child link="robot0/base_link"/>
   </joint>
-  <link name="target/t1"/>
-  <joint name="target/t1_joint" type="fixed">
-    <parent link="world"/>
-    <child link="target/t1"/>
-  </joint>
-  <xacro:s4_omni prefix="body0" parent="base_link" />
+  <xacro:s4_omni prefix="robot0/omni0" parent="robot0/base_link" />
   <!-- ===============  Gazebo =============== -->
   <gazebo>

Commit message: modify

File: s4_omni/urdf/s4_omni.urdf.xacro (robot description, xacro)
@@ -1,17 +1,6 @@
 <?xml version="1.0"?>
 <robot name="my_robo" xmlns:xacro="http://ros.org/wiki/xacro">
-  <xacro:include filename="$(find s4_omni)/urdf/body.urdf.xacro"/>
   <xacro:include filename="$(find s4_omni)/urdf/wheel.urdf.xacro"/>
   <xacro:macro name="s4_omni" params="prefix parent">
-<!--
-    <joint name="${prefix}_joint" type="floating">
-      <parent link="${parent}"/>
-      <child link="${prefix}_target0_link"/>
-      <origin rpy="0 0 ${dir}" xyz="${0.106*cos(dir)} ${0.106*sin(dir)} 0.098"/>
-    </joint>
--->
-<!--
-    <xacro:body prefix="body0" parent="base_link" />
--->
     <xacro:omni_wheel prefix="${prefix}/wheel0" parent="${parent}" radius="0.075" dir="${pi/3}"   height="0.019" />
     <xacro:omni_wheel prefix="${prefix}/wheel1" parent="${parent}" radius="0.075" dir="${pi}"     height="0.019" />

File: s4_omni/urdf/wheel.urdf.xacro (robot description, xacro)
@@ -12,5 +12,5 @@
       <visual>
         <geometry>
-          <mesh filename="package://srs004host/urdf/barrel.stl" />
+          <mesh filename="package://s4_omni/stl/barrel.stl" />
         </geometry>
         <material name="black"/>
@@ -18,5 +18,5 @@
       <collision>
         <geometry>
-          <mesh filename="package://srs004host/urdf/barrel.stl" />
+          <mesh filename="package://s4_omni/stl/barrel.stl" />
         </geometry>
       </collision>
@@ -64,5 +64,5 @@
       <visual>
         <geometry>
-          <mesh filename="package://srs004host/urdf/motor.stl" />
+          <mesh filename="package://s4_omni/stl/motor.stl" />
         </geometry>
         <origin xyz="0 0 0" rpy="0 0 0"/>
@@ -84,5 +84,5 @@
       <visual>
         <geometry>
-          <mesh filename="package://srs004host/urdf/housing.stl" />
+          <mesh filename="package://s4_omni/stl/housing.stl" />
         </geometry>
         <origin xyz="0 0 0" rpy="0 0 0"/>
