Commit message: modify

File: s4_hitsensor/urdf/s4_hitsensor.urdf.xacro (robot description, xacro)
@@ -22,5 +22,5 @@
           <mesh filename="package://s4_hitsensor/stl/target_plate.stl" />
         </geometry>
-        <material name="gray"/>
+        <material name="dark_green"/>
       </visual>
     </link>

File: s4_launch/urdf/s4_robot.urdf.xacro (robot description, xacro)
@@ -1,4 +1,5 @@
 <?xml version="1.0"?>
 <robot name="my_robo" xmlns:xacro="http://ros.org/wiki/xacro">
+  <xacro:include filename="$(find s4_operate)/urdf/s4_body.urdf.xacro"/>
   <xacro:include filename="$(find s4_omni)/urdf/s4_omni.urdf.xacro"/>
   <xacro:include filename="$(find s4_gun)/urdf/s4_gun.urdf.xacro"/>
@@ -10,7 +11,8 @@
       <child link="${prefix}/base_link"/>
     </joint>
+    <xacro:s4_body      prefix="${prefix}/body0"      parent="${prefix}/base_link" pos_z="0.041"/>
     <xacro:s4_omni      prefix="${prefix}/omni0"      parent="${prefix}/base_link" />
-    <xacro:s4_gun       prefix="${prefix}/gun0"       parent="${prefix}/base_link" pos_x="0.010" pos_z="0.038" />
-    <xacro:s4_hitsensor prefix="${prefix}/hitsensor0" parent="${prefix}/base_link" radius="0.1" height="0.1" />
+    <xacro:s4_gun       prefix="${prefix}/gun0"       parent="${prefix}/base_link" pos_x="0.0" pos_z="0.079" />
+    <xacro:s4_hitsensor prefix="${prefix}/hitsensor0" parent="${prefix}/base_link" radius="0.106" height="0.079" />
   </xacro:macro>
   <!-- ===============  Gazebo =============== -->

File: s4_operate/urdf/common.urdf.xacro (robot description, xacro)
@@ -18,11 +18,5 @@
   </material>
   <material name="yellow">
-    <color rgba="1.0 1.0 0.0 2.5"/>
-  </material>
-  <material name="green">
-    <color rgba="0.0 1.0 0 2.5"/>
-  </material>
-  <material name="dark_green">
-    <color rgba="0.0 0.5 0 2.5"/>
+    <color rgba="0 1.0 1.0 2.5"/>
   </material>
 </robot>
