Commit message: s4_hitsensor: modify for multi robot

File: s4_hitsensor/urdf/common.urdf.xacro (robot description, xacro)
@@ -17,6 +17,15 @@
     <color rgba="1.0 0.5 0.5 2.5"/>
   </material>
-  <material name="yellow">
-    <color rgba="0 1.0 1.0 2.5"/>
+  <material name="green">
+    <color rgba="0 1.0 0 2.5"/>
+  </material>
+  <material name="dark_green">
+    <color rgba="0 0.5 0 2.5"/>
+  </material>
+  <material name="blue">
+    <color rgba="0 0 1.0 2.5"/>
+  </material>
+  <material name="wood">
+    <color rgba="0.9 0.9 0.5 2.5"/>
   </material>
 </robot>
