Commit message: each rviz: modify s4_launch: modify

File: s4_launch/urdf/s4_robot.urdf.xacro (robot description, xacro)
@@ -1,18 +1,14 @@
 <?xml version="1.0"?>
 <robot name="my_robo" xmlns:xacro="http://ros.org/wiki/xacro">
-  <xacro:include filename="$(find s4_operate)/urdf/s4_body.urdf.xacro"/>
+  <xacro:include filename="$(find s4_system)/urdf/s4_body.urdf.xacro"/>
   <xacro:include filename="$(find s4_omni)/urdf/s4_omni.urdf.xacro"/>
   <xacro:include filename="$(find s4_gun)/urdf/s4_gun.urdf.xacro"/>
   <xacro:include filename="$(find s4_hitsensor)/urdf/s4_hitsensor.urdf.xacro"/>
-  <xacro:macro name="s4_robot" params="prefix parent">
-    <link name="${prefix}/base_link"/>
-      <joint name="${prefix}/base_joint" type="fixed"><!--floating-->
-      <parent link="${parent}"/>
-      <child link="${prefix}/base_link"/>
-    </joint>
-    <xacro:s4_body      prefix="${prefix}/body0"      parent="${prefix}/base_link" pos_z="0.044"/>
-    <xacro:s4_omni      prefix="${prefix}/omni0"      parent="${prefix}/base_link" />
-    <xacro:s4_gun       prefix="${prefix}/gun0"       parent="${prefix}/base_link" pos_x="0.020" pos_z="0.082" />
-    <xacro:s4_hitsensor prefix="${prefix}/hitsensor0" parent="${prefix}/base_link" radius="0.106" height="0.082" />
+  <xacro:macro name="s4_robot">
+    <link name="base_link"/>
+    <xacro:s4_body      prefix="body0"      parent="base_link" pos_z="0.044"/>
+    <xacro:s4_omni      prefix="omni0"      parent="base_link" />
+    <xacro:s4_gun       prefix="gun0"       parent="base_link" pos_x="0.020" pos_z="0.082" />
+    <xacro:s4_hitsensor prefix="hitsensor0" parent="base_link" radius="0.106" height="0.082" />
   </xacro:macro>
   <!-- ===============  Gazebo =============== -->

File: s4_launch/urdf/single_robot.urdf.xacro (robot description, xacro)
@@ -3,7 +3,5 @@
   <xacro:include filename="$(find s4_launch)/urdf/common.urdf.xacro"/>
   <xacro:include filename="$(find s4_launch)/urdf/s4_robot.urdf.xacro"/>
-  <xacro:arg name="robot_name" default="robot0"/>
-  <link name="world"/>
-  <xacro:s4_robot prefix="$(arg robot_name)" parent="world" />
+  <xacro:s4_robot />
   <!-- ===============  Gazebo =============== -->
   <gazebo>
