Commit message: s4_system: first commit

File: s4_system/urdf/s4_body.urdf.xacro (robot description, xacro)
@@ -11,5 +11,5 @@
         <origin xyz="0 0 0" rpy="0 0 0"/>
         <geometry>
-          <mesh filename="package://s4_operate/stl/body.stl" />
+          <mesh filename="package://s4_system/stl/body.stl" />
         </geometry>
         <material name="gray"/>
@@ -29,5 +29,5 @@
         <origin xyz="0 0 0" rpy="0 0 0"/>
         <geometry>
-          <mesh filename="package://s4_operate/stl/battery.stl" />
+          <mesh filename="package://s4_system/stl/battery.stl" />
         </geometry>
         <material name="blue"/>
@@ -47,5 +47,5 @@
         <origin xyz="0 0 0" rpy="0 0 0"/>
         <geometry>
-          <mesh filename="package://s4_operate/stl/bridge.stl" />
+          <mesh filename="package://s4_system/stl/bridge.stl" />
         </geometry>
         <material name="gray"/>
@@ -65,5 +65,5 @@
         <origin xyz="0 0 0" rpy="0 0 0"/>
         <geometry>
-          <mesh filename="package://s4_operate/stl/camera.stl" />
+          <mesh filename="package://s4_system/stl/camera.stl" />
         </geometry>
         <material name="light_red"/>
