Commit message: s4: vive move first complete

File: s4_vive/urdf/world.urdf.xacro (robot description, xacro)
@@ -4,9 +4,4 @@
   <xacro:include filename="$(find s4_vive)/urdf/s4_vive.urdf.xacro"/>
   <link name="world" />
-  <link name="robot0/base_link" />
-  <joint name="robot0/base_joint" type="floating">
-    <parent link="world"/>
-    <child  link="robot0/base_link"/>
-  </joint>
   <xacro:s4_vive_controller prefix="vive0/controller0" parent="world" />
   <xacro:s4_vive_controller prefix="vive0/controller1" parent="world" />
