Commit message: add package and change

File: s4_description/xacro/s4_body.xacro (robot description, xacro)
@@ -16,5 +16,5 @@
       </visual>
       <inertial>
-        <mass value="0.130"/>
+        <mass value="0.500"/>
         <inertia ixx="0.0001" ixy="0" ixz="0" iyy="0.0001" iyz="0" izz="0.0001"/>
       </inertial>
@@ -102,5 +102,5 @@
       </visual>
       <inertial>
-        <mass value="0.190"/>
+        <mass value="0.500"/>
         <inertia ixx="0.001" ixy="0" ixz="0" iyy="0.001" iyz="0" izz="0.0001"/>
       </inertial>
@@ -191,4 +191,23 @@
     </joint>
     <link name="${prefix}/imu_link" />
+    <gazebo reference="${prefix}/imu_link">
+      <gravity>true</gravity>
+      <sensor name="imu_sensor" type="imu">
+        <always_on>true</always_on>
+        <update_rate>100</update_rate>
+        <visualize>true</visualize>
+        <topic>__default_topic__</topic>
+        <plugin filename="libgazebo_ros_imu_sensor.so" name="imu_plugin">
+          <topicName>${robot}/${prefix}/imu/data</topicName>
+          <bodyName>imu_link</bodyName>
+          <updateRateHZ>10.0</updateRateHZ>
+          <gaussianNoise>0.0</gaussianNoise>
+          <xyzOffset>0 0 0</xyzOffset>
+          <rpyOffset>0 ${radians(180)} ${radians(-90)}</rpyOffset>
+          <frameName>${robot}/${prefix}/imu_link</frameName>
+        </plugin>
+        <pose>0 0 0 0 0 0</pose>
+      </sensor>
+    </gazebo>
   </xacro:macro>
 </robot>

File: s4_description/xacro/s4_targets.xacro (robot description, xacro)
@@ -2,4 +2,9 @@
 <robot xmlns:xacro="http://ros.org/wiki/xacro">
   <xacro:macro name="s4_target" params="prefix parent xyz rpy">
+    <joint name="${prefix}/frame_joint" type="fixed">
+      <parent link="${parent}"/>
+      <child  link="${prefix}/frame_link"/>
+      <origin rpy="${rpy}" xyz="${xyz}"/>
+    </joint>
     <link name="${prefix}/frame_link">
       <visual>
@@ -11,8 +16,8 @@
       </visual>
     </link>
-    <joint name="${prefix}/frame_joint" type="fixed"><!--floating-->
-      <parent link="${parent}"/>
-      <child  link="${prefix}/frame_link"/>
-      <origin rpy="${rpy}" xyz="${xyz}"/>
+    <joint name="${prefix}/plate_joint" type="fixed">
+      <parent link="${prefix}/frame_link"/>
+      <child  link="${prefix}/plate_link"/>
+      <origin rpy="0 0 0" xyz="0 0 0.06"/>
     </joint>
     <link name="${prefix}/plate_link">
@@ -28,9 +33,4 @@
       <material>Gazebo/Green</material>
     </gazebo>
-    <joint name="${prefix}/plate_joint" type="fixed"><!--floating-->
-      <parent link="${prefix}/frame_link"/>
-      <child  link="${prefix}/plate_link"/>
-      <origin rpy="0 0 0" xyz="0 0 0.06"/>
-    </joint>
   </xacro:macro>
   <xacro:macro name="s4_targets" params="prefix parent radius height">

File: s4_description/xacro/wheel.xacro (robot description, xacro)
@@ -2,5 +2,5 @@
 <robot xmlns:xacro="http://ros.org/wiki/xacro">
   <xacro:macro name="barrel" params="prefix parent dir">
-    <joint name="${prefix}_joint" type="fixed"><!--continuous-->
+    <joint name="${prefix}_joint" type="continuous">
       <parent link="${parent}"/>
       <child link="${prefix}_link"/>
@@ -26,12 +26,34 @@
       </inertial>
     </link>
-    <!-- ===============  Gazebo =============== -->
+    <transmission name="${prefix}_trans">
+      <type>transmission_interface/SimpleTransmission</type>
+      <joint name="${prefix}_joint">
+        <hardwareInterface>hardware_interface/EffortJointInterface</hardwareInterface>
+      </joint>
+      <actuator name="${prefix}_motor">
+        <hardwareInterface>hardware_interface/EffortJointInterface</hardwareInterface>
+        <mechanicalReduction>1</mechanicalReduction>
+      </actuator>
+    </transmission>
     <gazebo reference="${prefix}_link">
-      <mu1 value="3.0" />
-      <mu2 value="3.0" />
-      <kp value="10000" />
+      <mu1 value="2.5" />
+      <mu2 value="2.5" />
+      <kp value="1000" />
       <kd value="10" />
       <material>Gazebo/Black</material>
     </gazebo>
+    <joint name="${prefix}_mark_joint" type="fixed">
+      <parent link="${prefix}_link"/>
+      <child link="${prefix}_mark_link"/>
+      <origin rpy="0 0 0" xyz="0.005 0 0"/>
+    </joint>
+    <link name="${prefix}_mark_link">
+      <visual>
+        <geometry>
+          <box size="0.005 0.005 0.005"/>
+        </geometry>
+        <material name="white"/>
+      </visual>
+    </link>
     <gazebo reference="${prefix}_mark_link">
       <material>Gazebo/White</material>
@@ -62,5 +84,5 @@
       <origin rpy="0 ${radians(90)} 0" xyz="0.0227 0 0"/>
       <axis xyz="0 0 1"/>
-      <limit velocity="12.0" effort="10.0" />
+      <limit velocity="12.0" effort="1.0" />
       <dynamics damping="0.1"/>
     </joint>
@@ -74,5 +96,5 @@
       </visual>
       <inertial>
-        <mass value="0.009"/>
+        <mass value="0.003"/>
         <inertia ixx="0.0001" ixy="0" ixz="0" iyy="0.0001" iyz="0" izz="0.0001"/>
       </inertial>
@@ -86,5 +108,5 @@
       <inertial>
         <mass value="0.001"/>
-        <inertia ixx="0" ixy="0" ixz="0" iyy="0" iyz="0" izz="0.00001"/>
+        <inertia ixx="0.0001" ixy="0" ixz="0" iyy="0.0001" iyz="0" izz="0.0001"/>
       </inertial>
     </link>

Commit message: s4_description: modify

File: s4_description/xacro/s4_body.xacro (robot description, xacro)
@@ -19,4 +19,9 @@
         <inertia ixx="0.0001" ixy="0" ixz="0" iyy="0.0001" iyz="0" izz="0.0001"/>
       </inertial>
+      <collision>
+        <geometry>
+          <cylinder length="0.01" radius="0.1" />
+        </geometry>
+      </collision>
     </link>
     <joint name="${prefix}/lidar_joint" type="fixed">

File: s4_description/xacro/wheel.xacro (robot description, xacro)
@@ -22,6 +22,6 @@
       </collision>
       <inertial>
-        <mass value="0.001"/>
-        <inertia ixx="0.0001" ixy="0" ixz="0" iyy="0.0001" iyz="0" izz="0.0001"/>
+        <mass value="0.002"/>
+        <inertia ixx="0.000001" ixy="0" ixz="0" iyy="0.000001" iyz="0" izz="0.000001"/>
       </inertial>
     </link>
@@ -78,4 +78,9 @@
         <inertia ixx="0.0001" ixy="0" ixz="0" iyy="0.0001" iyz="0" izz="0.0001"/>
       </inertial>
+      <collision>
+        <geometry>
+          <mesh filename="package://s4_description/stl/motor.stl" />
+        </geometry>
+      </collision>
     </link>
     <joint name="${prefix}/wheel_joint" type="continuous">
@@ -88,4 +93,8 @@
     </joint>
     <link name="${prefix}/wheel_link">
+      <inertial>
+        <mass value="0.025"/>
+        <inertia ixx="0.0001" ixy="0" ixz="0" iyy="0.0001" iyz="0" izz="0.0001"/>
+      </inertial>
       <visual>
         <geometry>
@@ -95,8 +104,4 @@
         <material name="gray"/>
       </visual>
-      <inertial>
-        <mass value="0.003"/>
-        <inertia ixx="0.0001" ixy="0" ixz="0" iyy="0.0001" iyz="0" izz="0.0001"/>
-      </inertial>
     </link>
     <joint name="${prefix}/wheel_s_joint" type="fixed">
@@ -107,5 +112,5 @@
     <link name="${prefix}/wheel_s_link">
       <inertial>
-        <mass value="0.001"/>
+        <mass value="0.025"/>
         <inertia ixx="0.0001" ixy="0" ixz="0" iyy="0.0001" iyz="0" izz="0.0001"/>
       </inertial>

Commit message: before edit description

File: s4_description/xacro/s4_body.xacro (robot description, xacro)
@@ -8,4 +8,8 @@
     </joint>
     <link name="${prefix}/body_link">
+      <inertial>
+        <mass value="0.500"/>
+        <inertia ixx="0.0001" ixy="0" ixz="0" iyy="0.0001" iyz="0" izz="0.0001"/>
+      </inertial>
       <visual>
         <origin xyz="0 0 0" rpy="0 0 0"/>
@@ -15,64 +19,28 @@
         <material name="gray"/>
       </visual>
-      <inertial>
-        <mass value="0.500"/>
-        <inertia ixx="0.0001" ixy="0" ixz="0" iyy="0.0001" iyz="0" izz="0.0001"/>
-      </inertial>
       <collision>
+        <origin rpy="0 0 0" xyz="0 0 0.002"/>
         <geometry>
-          <cylinder length="0.01" radius="0.1" />
+          <cylinder radius="0.119" length="0.004" />
         </geometry>
       </collision>
     </link>
-    <joint name="${prefix}/lidar_joint" type="fixed">
+    <joint name="${prefix}/body2_joint" type="fixed">
       <parent link="${prefix}/body_link"/>
-      <child  link="${prefix}/lidar_link"/>
-      <origin rpy="0 0 ${radians(-90)}" xyz="0.075 0.010 0.030"/>
+      <child  link="${prefix}/body2_link"/>
+      <origin rpy="0 0 0" xyz="0 0 0.046"/>
     </joint>
-     <link name="${prefix}/lidar_link">
-      <visual>
-        <origin xyz="0 0 0" rpy="0 0 0"/>
+    <link name="${prefix}/body2_link">
+      <inertial>
+        <mass value="0.010"/>
+        <inertia ixx="0.00001" ixy="0" ixz="0" iyy="0.00001" iyz="0" izz="0.00001"/>
+      </inertial>
+      <collision>
+        <origin rpy="0 0 0" xyz="0 0 0.002"/>
         <geometry>
-          <mesh filename="package://s4_description/stl/ydlidar.stl" />
+          <cylinder radius="0.119" length="0.004" />
         </geometry>
-        <material name="light_blue"/>
-      </visual>
-      <inertial>
-        <mass value="0.130"/>
-        <inertia ixx="0.0001" ixy="0" ixz="0" iyy="0.0001" iyz="0" izz="0.0001"/>
-      </inertial>
+      </collision>
     </link>
-    <gazebo reference="${prefix}/lidar_link">
-      <material>Gazebo/Blue</material>
-      <sensor type="ray" name="head_lidar">
-        <pose>0 0 0 0 0 0</pose>
-        <visualize>false</visualize>
-        <update_rate>10</update_rate>
-        <ray>
-          <scan>
-            <horizontal>
-              <samples>400</samples>
-              <resolution>1</resolution>
-              <min_angle>-3.141592</min_angle>
-              <max_angle> 3.141592</max_angle>
-            </horizontal>
-          </scan>
-          <range>
-            <min>0.10</min>
-            <max>20.0</max>
-            <resolution>0.01</resolution>
-          </range>
-          <noise>
-            <type>gaussian</type>
-            <mean>0.0</mean>
-            <stddev>0.01</stddev>
-          </noise>
-        </ray>
-        <plugin name="gazebo_ros_lidar_controller" filename="libgazebo_ros_laser.so">
-          <topicName>${robot}/${prefix}/laser/scan</topicName>
-          <frameName>${robot}/${prefix}/lidar_link</frameName>
-        </plugin>
-      </sensor>
-    </gazebo>
     <joint name="${prefix}/battery_joint" type="fixed">
       <parent link="${prefix}/body_link"/>
@@ -111,65 +79,4 @@
       </inertial>
     </link>
-    <joint name="${prefix}/camera_joint" type="fixed">
-      <parent link="${prefix}/bridge_link"/>
-      <child  link="${prefix}/camera_link"/>
-      <origin rpy="${radians(-90)} 0 ${radians(-90)}" xyz="0.015 0 0.1601"/>
-    </joint>
-    <link name="${prefix}/camera_link">
-      <visual>
-        <origin xyz="0 0 0" rpy="0 0 0"/>
-        <geometry>
-          <mesh filename="package://s4_description/stl/camera.stl" />
-        </geometry>
-        <material name="light_blue"/>
-      </visual>
-      <inertial>
-        <mass value="0.190"/>
-        <inertia ixx="0.001" ixy="0" ixz="0" iyy="0.001" iyz="0" izz="0.0001"/>
-      </inertial>
-    </link>
-    <gazebo reference="${prefix}/camera_sim_link">
-      <material>Gazebo/Blue</material>
-      <sensor type="camera" name="camera1">
-        <update_rate>10.0</update_rate>
-        <camera name="head">
-          <horizontal_fov>1.3962634</horizontal_fov>
-          <image>
-            <width>800</width>
-            <height>600</height>
-            <format>R8G8B8</format>
-          </image>
-          <clip>
-            <near>0.02</near>
-            <far>300</far>
-          </clip>
-          <noise>
-            <type>gaussian</type>
-            <mean>0.0</mean>
-            <stddev>0.007</stddev>
-          </noise>
-        </camera>
-        <plugin name="camera_controller" filename="libgazebo_ros_camera.so">
-          <alwaysOn>true</alwaysOn>
-          <updateRate>10.0</updateRate>
-          <cameraName>${robot}/${prefix}/head_camera</cameraName>
-          <imageTopicName>image_raw</imageTopicName>
-          <cameraInfoTopicName>camera_info</cameraInfoTopicName>
-          <frameName>camera_link</frameName>
-          <hackBaseline>0.07</hackBaseline>
-          <distortionK1>0.0</distortionK1>
-          <distortionK2>0.0</distortionK2>
-          <distortionK3>0.0</distortionK3>
-          <distortionT1>0.0</distortionT1>
-          <distortionT2>0.0</distortionT2>
-        </plugin>
-      </sensor>
-    </gazebo>
-    <joint name="${prefix}/camera_sim_joint" type="fixed">
-      <parent link="${prefix}/camera_link"/>
-      <child  link="${prefix}/camera_sim_link"/>
-      <origin rpy="0 ${radians(-90)} ${radians(90)}" xyz="0 0 0"/>
-    </joint>
-    <link name="${prefix}/camera_sim_link"/>
     <joint name="${prefix}/tracker_joint" type="fixed">
       <parent link="${prefix}/bridge_link"/>
@@ -190,29 +97,4 @@
       </inertial>
     </link>
-    <joint name="${prefix}/imu_joint" type="fixed">
-      <parent link="${prefix}/bridge_link"/>
-      <child  link="${prefix}/imu_link"/>
-      <origin rpy="${radians(180)} 0 ${radians(90)}" xyz="-0.078 0 0.138"/>
-    </joint>
-    <link name="${prefix}/imu_link" />
-    <gazebo reference="${prefix}/imu_link">
-      <gravity>true</gravity>
-      <sensor name="imu_sensor" type="imu">
-        <always_on>true</always_on>
-        <update_rate>100</update_rate>
-        <visualize>true</visualize>
-        <topic>__default_topic__</topic>
-        <plugin filename="libgazebo_ros_imu_sensor.so" name="imu_plugin">
-          <topicName>${robot}/${prefix}/imu/data</topicName>
-          <bodyName>imu_link</bodyName>
-          <updateRateHZ>10.0</updateRateHZ>
-          <gaussianNoise>0.0</gaussianNoise>
-          <xyzOffset>0 0 0</xyzOffset>
-          <rpyOffset>0 ${radians(180)} ${radians(-90)}</rpyOffset>
-          <frameName>${robot}/${prefix}/imu_link</frameName>
-        </plugin>
-        <pose>0 0 0 0 0 0</pose>
-      </sensor>
-    </gazebo>
   </xacro:macro>
 </robot>

File: s4_description/xacro/s4_gun.xacro (robot description, xacro)
@@ -20,7 +20,4 @@
       </inertial>
     </link>
-    <gazebo reference="${prefix}/base1_link">
-      <material>Gazebo/Gray</material>
-    </gazebo>
     <joint name="${prefix}/base2_joint" type="continuous">
       <parent link="${prefix}/base1_link"/>
@@ -53,7 +50,4 @@
       </actuator>
     </transmission>
-    <gazebo reference="${prefix}/base2_link">
-      <material>Gazebo/Gray</material>
-    </gazebo>
     <joint name="${prefix}/gun_joint" type="continuous">
       <parent link="${prefix}/base2_link"/>

File: s4_description/xacro/s4_robot.xacro (robot description, xacro)
@@ -6,4 +6,5 @@
   <xacro:include filename="$(find s4_description)/xacro/s4_omni.xacro"/>
   <xacro:include filename="$(find s4_description)/xacro/s4_gun.xacro"/>
+  <xacro:include filename="$(find s4_description)/xacro/s4_sensor.xacro"/>
   <xacro:include filename="$(find s4_description)/xacro/s4_targets.xacro"/>
   <xacro:macro name="s4_robot">
@@ -12,4 +13,5 @@
     <xacro:s4_omni      prefix="omni0"    parent="base_link" />
     <xacro:s4_gun       prefix="gun0"     parent="base_link" pos_x="0.020" pos_z="0.094" />
+    <xacro:s4_sensor    prefix="sensor0"  parent="base_link" ns="$(arg robot)"/>
     <xacro:s4_targets   prefix="targets0" parent="base_link" radius="0.106" height="0.094"/>
   </xacro:macro>

File: s4_description/xacro/wheel.xacro (robot description, xacro)
@@ -39,5 +39,5 @@
       <mu1 value="2.5" />
       <mu2 value="2.5" />
-      <kp value="1000" />
+      <kp value="5000" />
       <kd value="10" />
       <material>Gazebo/Black</material>
@@ -61,6 +61,35 @@
   </xacro:macro>
   <xacro:macro name="omni_wheel" params="prefix parent radius dir height">
+    <joint name="${prefix}/sus_joint" type="prismatic">
+      <parent link="${parent}"/>
+      <child  link="${prefix}/sus_link"/>
+      <limit lower="-0.02" upper="0.02" effort="100" velocity="1.0" />
+      <axis xyz="0 0 1"/>
+      <origin xyz="0 0 0" rpy="0 0 0"/>
+      <dynamics damping="0.7"/>
+    </joint>
+    <transmission name="${prefix}/sus_trans">
+      <type>transmission_interface/SimpleTransmission</type>
+      <joint name="${prefix}/sus_joint">
+          <hardwareInterface>hardware_interface/EffortJointInterface</hardwareInterface>
+      </joint>
+      <actuator name="${prefix}/sus_motor">
+        <hardwareInterface>hardware_interface/EffortJointInterface</hardwareInterface>
+        <mechanismReduction>1</mechanismReduction>
+      </actuator>
+    </transmission>
+    <gazebo reference="${prefix}/sus_joint">
+      <kp>50000</kp>
+      <kd>500</kd>
+    </gazebo>
+    <link name="${prefix}/sus_link">
+      <inertial>
+        <mass value="1.0"/>
+        <origin xyz="0 0 0.25" rpy="0 0 0"/>
+        <inertia ixx="0.01" ixy="0.0" ixz="0.0" iyy="0.01" iyz="0.0" izz="0.01"/>
+      </inertial>
+    </link>
     <joint name="${prefix}/motor_joint" type="fixed">
-      <parent link="${parent}"/>
+      <parent link="${prefix}/sus_link"/>
       <child link="${prefix}/motor_link"/>
       <origin rpy="0 0 ${dir}" xyz="${radius*cos(dir)} ${radius*sin(dir)} ${height}"/>
@@ -79,6 +108,7 @@
       </inertial>
       <collision>
+        <origin rpy="0 ${radians(90)} 0" xyz="-0.025 0 0"/>
         <geometry>
-          <mesh filename="package://s4_description/stl/motor.stl" />
+          <cylinder radius="0.012" length="0.05" />
         </geometry>
       </collision>
@@ -89,5 +119,5 @@
       <origin rpy="0 ${radians(90)} 0" xyz="0.0227 0 0"/>
       <axis xyz="0 0 1"/>
-      <limit velocity="12.0" effort="1.0" />
+      <limit velocity="40.0" effort="3.0" />
       <dynamics damping="0.1"/>
     </joint>
@@ -116,12 +146,12 @@
       </inertial>
     </link>
-    <xacro:barrel prefix="${prefix}/barrel_1" parent="${prefix}/wheel_link" dir="0"/>
-    <xacro:barrel prefix="${prefix}/barrel_2" parent="${prefix}/wheel_link" dir="${pi/2}"/>
-    <xacro:barrel prefix="${prefix}/barrel_3" parent="${prefix}/wheel_link" dir="${pi}"/>
-    <xacro:barrel prefix="${prefix}/barrel_4" parent="${prefix}/wheel_link" dir="${-pi/2}"/>
-    <xacro:barrel prefix="${prefix}/barrel_5" parent="${prefix}/wheel_s_link" dir="0"/>
-    <xacro:barrel prefix="${prefix}/barrel_6" parent="${prefix}/wheel_s_link" dir="${pi/2}"/>
-    <xacro:barrel prefix="${prefix}/barrel_7" parent="${prefix}/wheel_s_link" dir="${pi}"/>
-    <xacro:barrel prefix="${prefix}/barrel_8" parent="${prefix}/wheel_s_link" dir="${-pi/2}"/>
+    <xacro:barrel prefix="${prefix}/barrel_0" parent="${prefix}/wheel_link" dir="0"/>
+    <xacro:barrel prefix="${prefix}/barrel_1" parent="${prefix}/wheel_link" dir="${pi/2}"/>
+    <xacro:barrel prefix="${prefix}/barrel_2" parent="${prefix}/wheel_link" dir="${pi}"/>
+    <xacro:barrel prefix="${prefix}/barrel_3" parent="${prefix}/wheel_link" dir="${-pi/2}"/>
+    <xacro:barrel prefix="${prefix}/barrel_4" parent="${prefix}/wheel_s_link" dir="0"/>
+    <xacro:barrel prefix="${prefix}/barrel_5" parent="${prefix}/wheel_s_link" dir="${pi/2}"/>
+    <xacro:barrel prefix="${prefix}/barrel_6" parent="${prefix}/wheel_s_link" dir="${pi}"/>
+    <xacro:barrel prefix="${prefix}/barrel_7" parent="${prefix}/wheel_s_link" dir="${-pi/2}"/>
     <!-- ===============  Transmission =============== -->
     <transmission name="${prefix}/wheel_trans">
@@ -139,10 +169,8 @@
       <mu1 value="0.8" />
       <mu2 value="0.8" />
-      <material>Gazebo/Gray</material>
     </gazebo>
     <gazebo reference="${prefix}/motor_link">
       <mu1 value="0.8" />
       <mu2 value="0.8" />
-      <material>Gazebo/Gray</material>
     </gazebo>
   </xacro:macro>
