Commit message: s4_description: modify

File: s4_description/xacro/s4_body.xacro (robot description, xacro)
@@ -1,5 +1,5 @@
 <?xml version="1.0"?>
 <robot xmlns:xacro="http://ros.org/wiki/xacro">
-  <xacro:macro name="s4_body" params="prefix robot parent pos_z">
+  <xacro:macro name="s4_body" params="prefix parent pos_z">
     <joint name="${prefix}/body_joint" type="fixed">
       <parent link="${parent}"/>

File: s4_description/xacro/s4_robot.xacro (robot description, xacro)
@@ -1,6 +1,6 @@
 <?xml version="1.0"?>
-<robot name="my_robo" xmlns:xacro="http://ros.org/wiki/xacro">
-  <xacro:arg name="robot" default="default_robot"/>
-  <xacro:include filename="$(find s4_description)/xacro/common.xacro"/>
+<robot name="robot" xmlns:xacro="http://ros.org/wiki/xacro">
+  <xacro:arg name="robot_name" default="default_robot"/>
+  <xacro:include filename="$(find s4_description)/xacro/material.xacro"/>
   <xacro:include filename="$(find s4_description)/xacro/s4_body.xacro"/>
   <xacro:include filename="$(find s4_description)/xacro/s4_omni.xacro"/>
@@ -10,8 +10,8 @@
   <xacro:macro name="s4_robot">
     <link name="base_link"/>
-    <xacro:s4_body      prefix="body0"    parent="base_link" robot="$(arg robot)" pos_z="0.044"/>
+    <xacro:s4_body      prefix="body0"    parent="base_link"  pos_z="0.044"/>
     <xacro:s4_omni      prefix="omni0"    parent="base_link" />
     <xacro:s4_gun       prefix="gun0"     parent="base_link" pos_x="0.020" pos_z="0.094" />
-    <xacro:s4_sensor    prefix="sensor0"  parent="base_link" ns="$(arg robot)"/>
+    <xacro:s4_sensor    prefix="sensor0"  parent="base_link" robot_name="$(arg robot_name)"/>
     <xacro:s4_targets   prefix="targets0" parent="base_link" radius="0.106" height="0.094"/>
   </xacro:macro>
@@ -20,5 +20,5 @@
   <gazebo>
     <plugin name="gazebo_ros_control" filename="libgazebo_ros_control.so">
-      <robotNamespace>$(arg robot)</robotNamespace>
+      <robotNamespace>$(arg robot_name)</robotNamespace>
     </plugin>
   </gazebo>

File: s4_description/xacro/s4_sensor.xacro (robot description, xacro)
@@ -1,5 +1,5 @@
 <?xml version="1.0"?>
 <robot xmlns:xacro="http://ros.org/wiki/xacro">
-  <xacro:macro name="s4_sensor" params="prefix parent ns">
+  <xacro:macro name="s4_sensor" params="prefix parent robot_name">
     <joint name="${prefix}/camera_joint" type="fixed">
       <parent link="${parent}"/>
@@ -23,14 +23,9 @@
       <material>Gazebo/Blue</material>
     </gazebo>
-    <joint name="${prefix}/camera_sim_joint" type="fixed">
-      <parent link="${prefix}/head_camera_link"/>
-      <child  link="${prefix}/head_camera_sim_link"/>
-      <origin rpy="0 ${radians(-90)} ${radians(90)}" xyz="0 0 0"/>
-    </joint>
-    <link name="${prefix}/head_camera_sim_link"/>
-    <gazebo reference="${prefix}/head_camera_sim_link">
-      <sensor type="camera" name="camera1">
+    <gazebo reference="${prefix}/head_camera_link">
+      <sensor type="camera" name="head_camera">
         <update_rate>10.0</update_rate>
-        <camera name="head">
+        <camera name="head_camera">
+          <pose>0 0 0 0 ${radians(-90)} ${radians(90)}</pose>
           <horizontal_fov>1.3962634</horizontal_fov>
           <image>
@@ -52,8 +47,8 @@
           <alwaysOn>true</alwaysOn>
           <updateRate>10.0</updateRate>
-          <cameraName>${ns}/${prefix}/head_camera</cameraName>
+          <cameraName>device/${prefix}/head_camera</cameraName>
           <imageTopicName>image_raw</imageTopicName>
           <cameraInfoTopicName>camera_info</cameraInfoTopicName>
-          <frameName>camera_link</frameName>
+          <frameName>${prefix}/head_camera_link</frameName>
           <hackBaseline>0.07</hackBaseline>
           <distortionK1>0.0</distortionK1>
@@ -65,10 +60,10 @@
       </sensor>
     </gazebo>
-    <joint name="${prefix}/front_lidar_joint" type="fixed">
+    <joint name="${prefix}/front_laser_joint" type="fixed">
       <parent link="${parent}"/>
-      <child  link="${prefix}/front_lidar_link"/>
+      <child  link="${prefix}/front_laser_link"/>
       <origin rpy="0 0 ${radians(-90)}" xyz="0.075 0.010 0.074"/>
     </joint>
-    <link name="${prefix}/front_lidar_link">
+    <link name="${prefix}/front_laser_link">
       <visual>
         <origin xyz="0 0 0" rpy="0 0 0"/>
@@ -83,7 +78,7 @@
       </inertial>
     </link>
-    <gazebo reference="${prefix}/front_lidar_link">
+    <gazebo reference="${prefix}/front_laser_link">
       <material>Gazebo/Blue</material>
-      <sensor type="ray" name="front_lidar">
+      <sensor type="ray" name="front_laser">
         <pose>0 0 0 0 0 0</pose>
         <visualize>false</visualize>
@@ -110,6 +105,6 @@
         </ray>
         <plugin name="gazebo_ros_lidar_controller" filename="libgazebo_ros_laser.so">
-          <topicName>${ns}/${prefix}/front_lidar/scan</topicName>
-          <frameName>${ns}/${prefix}/front_lidar_link</frameName>
+          <topicName>device/${prefix}/front_laser/scan</topicName>
+          <frameName>${prefix}/front_laser_link</frameName>
         </plugin>
       </sensor>
@@ -138,5 +133,5 @@
         <topic>__default_topic__</topic>
         <plugin filename="libgazebo_ros_imu_sensor.so" name="imu_plugin">
-          <topicName>${ns}/${prefix}/imu/data</topicName>
+          <topicName>device/${prefix}/imu/data</topicName>
           <bodyName>imu_link</bodyName>
           <updateRateHZ>10.0</updateRateHZ>
@@ -144,5 +139,5 @@
           <xyzOffset>0 0 0</xyzOffset>
           <rpyOffset>0 ${radians(180)} ${radians(-90)}</rpyOffset>
-          <frameName>${ns}/${prefix}/imu_link</frameName>
+          <frameName>${robot_name}/${prefix}/imu_link</frameName>
         </plugin>
         <pose>0 0 0 0 0 0</pose>
