Commit message: modify

File: s4_description/xacro/s4_sensor.xacro (robot description, xacro)
@@ -28,5 +28,5 @@
         <camera name="head_camera">
           <pose>0 0 0 0 ${radians(-90)} ${radians(90)}</pose>
-          <horizontal_fov>1.3962634</horizontal_fov>
+          <horizontal_fov>1.58</horizontal_fov>
           <image>
             <width>800</width>
@@ -51,10 +51,10 @@
           <cameraInfoTopicName>camera_info</cameraInfoTopicName>
           <frameName>${prefix}/head_camera_link</frameName>
-          <hackBaseline>0.07</hackBaseline>
-          <distortionK1>0.0</distortionK1>
-          <distortionK2>0.0</distortionK2>
-          <distortionK3>0.0</distortionK3>
-          <distortionT1>0.0</distortionT1>
-          <distortionT2>0.0</distortionT2>
+          <hackBaseline>0.0</hackBaseline>
+          <distortionK1> 0.016</distortionK1>
+          <distortionK2>-0.026</distortionK2>
+          <distortionK3> 0.000</distortionK3>
+          <distortionT1> 0.002</distortionT1>
+          <distortionT2> 0.004</distortionT2>
         </plugin>
       </sensor>
@@ -113,7 +113,7 @@
       <parent link="${parent}"/>
       <origin rpy="${radians(180)} 0 ${radians(90)}" xyz="${-0.078+0.005} 0 ${0.138+0.094}"/>
-      <child  link="${prefix}/imu_link"/>
+      <child  link="${prefix}/imu0_link"/>
     </joint>
-    <link name="${prefix}/imu_link">
+    <link name="${prefix}/imu0_link">
       <visual>
         <origin xyz="0 0 0" rpy="0 0 0"/>
@@ -124,5 +124,5 @@
       </visual>
     </link>
-    <gazebo reference="${prefix}/imu_link">
+    <gazebo reference="${prefix}/imu0_link">
       <material>Gazebo/Blue</material>
       <gravity>true</gravity>
@@ -133,11 +133,11 @@
         <topic>__default_topic__</topic>
         <plugin filename="libgazebo_ros_imu_sensor.so" name="imu_plugin">
-          <topicName>device/${prefix}/imu/data</topicName>
-          <bodyName>imu_link</bodyName>
+          <topicName>device/${prefix}/imu0/data</topicName>
+          <bodyName>imu0_link</bodyName>
           <updateRateHZ>10.0</updateRateHZ>
           <gaussianNoise>0.0</gaussianNoise>
           <xyzOffset>0 0 0</xyzOffset>
           <rpyOffset>0 ${radians(180)} ${radians(-90)}</rpyOffset>
-          <frameName>${robot_name}/${prefix}/imu_link</frameName>
+          <frameName>${robot_name}/${prefix}/imu0_link</frameName>
         </plugin>
         <pose>0 0 0 0 0 0</pose>

Commit message: s4_description: modify

File: s4_description/xacro/s4_sensor.xacro (robot description, xacro)
@@ -112,5 +112,5 @@
     <joint name="${prefix}/imu_joint" type="fixed">
       <parent link="${parent}"/>
-      <origin rpy="${radians(180)} 0 ${radians(90)}" xyz="${-0.078+0.005} 0 ${0.138+0.094}"/>
+      <origin rpy="0 0 ${radians(-90)}" xyz="-0.03 0 0.28"/>
       <child  link="${prefix}/imu0_link"/>
     </joint>

Commit message: s4_description: modify

File: s4_description/xacro/s4_sensor.xacro (robot description, xacro)
@@ -144,4 +144,23 @@
       </sensor>
     </gazebo>
+    <!-- for range -->
+    <joint name="${prefix}/range0_joint" type="fixed">
+      <parent link="${parent}"/>
+      <origin rpy="0 0 ${radians(159)}" xyz="-0.085 0.061 0.104"/>
+      <child  link="${prefix}/range0_link"/>
+    </joint>
+    <link name="${prefix}/range0_link"/>
+     <joint name="${prefix}/range1_joint" type="fixed">
+      <parent link="${parent}"/>
+      <origin rpy="0 0 ${radians(180)}" xyz="-0.105 0.0 0.074"/>
+      <child  link="${prefix}/range1_link"/>
+    </joint>
+    <link name="${prefix}/range1_link"/>
+    <joint name="${prefix}/range2_joint" type="fixed">
+      <parent link="${parent}"/>
+      <origin rpy="0 0 ${radians(-159)}" xyz="-0.085 -0.061 0.104"/>
+      <child  link="${prefix}/range2_link"/>
+    </joint>
+    <link name="${prefix}/range2_link"/>
   </xacro:macro>
 </robot>
